Commit message: add all changes

File: packages/irb120/ros2srrc_irb120_gazebo/urdf/irb120.urdf.xacro (robot description, xacro)
@@ -50,6 +50,5 @@
     <gazebo>
       <plugin filename="libgazebo_ros2_control.so" name="gazebo_ros2_control">
-        <robot_sim_type>gazebo_ros2_control/GazeboSystem</robot_sim_type>
-        <!-- IRB120 Controller -->
+        <robot_sim_type>gz_ros2_control/GazeboSimSystem</robot_sim_type>
         <parameters>$(find ros2srrc_robots)/irb120/config/controller.yaml</parameters>
       </plugin>

File: ros2srrc_robots/irb120/urdf/irb120_macro.urdf.xacro (robot description, xacro)
@@ -37,5 +37,5 @@
 #  COPYRIGHT - ROS-Industrial                                                           #
 #  (ORIGINAL LICENSE) -> Licensed under the Apache-2.0 License.                         #
-#                                                                                       #
+#                     abb_table                                                                  #
 #  CHANGES MADE:                                                                        #
 #  The original files contain the .urdf information of the robot for ROS1, and these    #
@@ -277,4 +277,13 @@
       <dynamics damping="1.0" friction="1.0"/>
     </joint>
+    <!-- joint_6 modified -->
+     <!-- <joint name="joint_6" type="revolute">
+      <origin rpy="0 0 0" xyz="0.072 0 0"/>
+      <parent link="link_5"/>
+      <child link="link_6"/>
+      <limit effort="1000" lower="-3.14" upper="3.14" velocity="7.33038"/>
+      <axis xyz="1 0 0"/>
+      <dynamics damping="1.0" friction="1.0"/>
+    </joint> -->
     <!-- end of joint list -->
     <!-- ROS-Industrial 'base' frame: base_link to ABB World Coordinates transform -->

File: ros2srrc_robots/irb120/urdf/irb120_ros2control.xacro (robot description, xacro)
@@ -51,21 +51,21 @@
     <!-- 1. ROS2_CONTROL tag name: -->
     <!-- A. GAZEBO SIMULATION: -->
-    <xacro:unless value="${bringup}">
-      <xacro:property name="name" value="GazeboSystem"/>
-    </xacro:unless>
+    <!-- <xacro:unless value="${bringup}"> -->
+      <!-- <xacro:property name="name" value="GazeboSimSystem"/> -->
+    <!-- </xacro:unless> -->
     <!-- B. ROBOT BRINGUP: -->
-    <xacro:if value="${bringup}">
-      <xacro:property name="name" value="ABBMultiInterfaceHardware"/>
-    </xacro:if>
+    <!-- <xacro:if value="${bringup}"> -->
+    <xacro:property name="name" value="ABBMultiInterfaceHardware"/>
+    <!-- </xacro:if> -->
     <!-- 3. Load ROS2_CONTROL: -->
     <ros2_control name="${name}" type="system">
       <!-- A. GAZEBO SIMULATION: -->
-      <xacro:unless value="${bringup}">
+      <!-- <xacro:unless value="${bringup}">
         <hardware>
-          <plugin>gazebo_ros2_control/GazeboSystem</plugin>
+          <plugin>gz_ros2_control/GazeboSimSystem</plugin>
         </hardware>
-      </xacro:unless>
+      </xacro:unless> -->
       <!-- B. ROBOT BRINGUP: -->
-      <xacro:if value="${bringup}">
+      <!-- <xacro:if value="${bringup}"> -->
         <hardware>
           <plugin>abb_hardware_interface/ABBSystemHardware</plugin>
@@ -74,5 +74,5 @@
           <param name="egm_port">6511</param>
         </hardware>
-      </xacro:if>
+      <!-- </xacro:if> -->
       <!-- irb120_joint1 -->
       <joint name="joint_1">
@@ -138,5 +138,5 @@
       <joint name="joint_5">
         <command_interface name="position">
-          <param name="min">-2.00</param>       <!-- Joint5 limits lowered to +-2rad -->
+          <param name="min">-2.00</param>
           <param name="max">2.00</param>
         </command_interface>
@@ -146,5 +146,5 @@
         </command_interface>
         <state_interface name="position">
-          <param name="initial_value">1.570796</param>
+          <param name="initial_value">0.0</param>
         </state_interface>
         <state_interface name="velocity"/>
@@ -168,5 +168,5 @@
       <xacro:unless value="${bringup}">
         <xacro:if value="${EE}">
-          <xacro:include filename="$(find ros2srrc_endeffectors)/${EE_name}/urdf/${EE_name}_ros2control.xacro" />
+          <xacro:include filename="$(find my_new_GRIPPER_package)/${EE_name}/urdf/${EE_name}_ros2control.xacro" />
           <xacro:EE_ros2control />
         </xacro:if>
